File: Hardware/Project_Milestone04_PCB.brd (EAGLE design)
At the start: 193 x 107.6 mm, 10 parts, among them IC2 7805T

Commit message: pcb updated
Parts:
- moved C2 61.4 mm to (55.9, 63.5)
- moved R2 54.9 mm to (73.7, 73.7)
- moved C3 51.4 mm to (61.0, 48.3)
- moved IC2 51.4 mm to (58.4, 20.3)
- moved C4 38.1 mm to (63.5, 73.7)
- moved S1 30.9 mm to (66.0, 88.9)
- moved LED2 20.9 mm to (71.1, 48.3)
- moved R1 20.5 mm to (72.4, 57.1)
- moved G1 14.8 mm to (77.5, 26.7)
Routing:
- net N$7: track 101.3 -> 53.0 mm
- net N$1: track 98.6 -> 52.6 mm
- net VCC: track 220.6 -> 190.6 mm
- net N$4: track 24.1 -> 9.94 mm
- net N$2: track 23.1 -> 14.8 mm
- net GND: track 3.66 -> 4.66 mm
Other:
- board size 193 x 107.6 mm -> 134.6 x 107.6 mm
